File: pico506.kicad_pcb (KiCad board)
At the start: 2 copper layers, 138 x 79 mm, 62 parts, among them J1 ST-506 CONTROL, J2 ST-506 DATA, J3 AMP 350211-1, J4 DRIVE SELECT, J5 UART, J6 SERVO GATE 3V3, J7 FRONT LED, Q1 2N3904, SW1 RESET, U1 Raspberry Pi Pico, U2 74LS05, U3 74LS05, U4 7438, U5 7438, U6 AM26LS31CN, U7 MC3486N

Commit message: Point silkscreen at this repo, credit upstream firmware
Other:
- board text added: "FIRMWARE: github.com/kuba2k2/pico506"
- board text added: "github.com/hmerrett/pico506-pcb"
- board text removed: "github.com/kuba2k2/pico506"
Changed lines of the file:
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@@
 			)
 		)
-		(fp_text user "K"
-			(at 0 -2.1 0)
+		(fp_text user "${REFERENCE}"
+			(at 5.47 0 0)
 			(layer "F.Fab")
 			(effects
@@
 			)
 		)
-		(fp_text user "${REFERENCE}"
-			(at 5.47 0 0)
+		(fp_text user "K"
+			(at 0 -2.1 0)
 			(layer "F.Fab")
 			(effects
@@
 			(layer "F.Fab")
 		)
-		(fp_text user "1"
-			(at -11.43 -7.38 0)
+		(fp_text user "19"
+			(at 11.43 -7.38 0)
 			(layer "F.SilkS")
 			(effects
@@
 			)
 		)
-		(fp_text user "19"
-			(at 11.43 -7.38 0)
+		(fp_text user "1"
+			(at -11.43 -7.38 0)
 			(layer "F.SilkS")
 			(effects
@@
 			)
 		)
-		(fp_text user "20"
-			(at 11.43 -7.38 0)
+		(fp_text user "2"
+			(at -11.43 -7.38 0)
 			(layer "B.SilkS")
 			(effects
@@
 			)
 		)
-		(fp_text user "2"
-			(at -11.43 -7.38 0)
+		(fp_text user "20"
+			(at 11.43 -7.38 0)
 			(layer "B.SilkS")
 			(effects
@@
 			(layer "F.Fab")
 		)
-		(fp_text user "1:+12V"
-			(at -7.62 -2.7 0)
+		(fp_text user "4:+5V"
+			(at 7.62 -2.7 0)
 			(layer "F.SilkS")
 			(effects
@@
 			)
 		)
-		(fp_text user "4:+5V"
-			(at 7.62 -2.7 0)
+		(fp_text user "1:+12V"
+			(at -7.62 -2.7 0)
 			(layer "F.SilkS")
 			(effects
@@
 		(layer "Edge.Cuts")
 	)
-	(gr_text "+12V"
-		(at 53 74.6 0)
+	(gr_text "PWR"
+		(at 31.6 56 90)
 		(layer "F.SilkS")
 		(effects
@@
 		)
 	)
-	(gr_text "J1 CONTROL"
-		(at 84.1 96.3 0)
+	(gr_text "GND SG"
+		(at 86.7 31.2 0)
 		(layer "F.SilkS")
 		(effects
 			(font
-				(size 1 1)
-				(thickness 0.15)
+				(size 0.8 0.8)
+				(thickness 0.12)
 			)
 		)
 	)
-	(gr_text "WF EN"
-		(at 94.7 31.2 0)
+	(gr_text "+12V"
+		(at 53 74.6 0)
 		(layer "F.SilkS")
 		(effects
@@
 		)
 	)
-	(gr_text "J2 DATA"
-		(at 151.45 96.3 0)
+	(gr_text "J1 CONTROL"
+		(at 84.1 96.3 0)
 		(layer "F.SilkS")
 		(effects
@@
 		)
 	)
-	(gr_text "RX TX GND"
-		(at 73.5 31.2 0)
+	(gr_text "TERM: LAST DRIVE ONLY"
+		(at 42 89.5 0)
 		(layer "F.SilkS")
 		(effects
 			(font
-				(size 0.8 0.8)
-				(thickness 0.12)
+				(size 0.9 0.9)
+				(thickness 0.135)
 			)
 		)
@@
 		)
 	)
-	(gr_text "LED"
-		(at 51.5 34 0)
+	(gr_text "-  +"
+		(at 54.7 31.4 0)
 		(layer "F.SilkS")
 		(effects
@@
 		)
 	)
-	(gr_text "-  +"
-		(at 54.7 31.4 0)
+	(gr_text "WF EN"
+		(at 94.7 31.2 0)
 		(layer "F.SilkS")
 		(effects
@@
 		)
 	)
-	(gr_text "GND SG"
-		(at 86.7 31.2 0)
+	(gr_text "RX TX GND"
+		(at 73.5 31.2 0)
 		(layer "F.SilkS")
 		(effects
@@
 		)
 	)
-	(gr_text "RST"
-		(at 160.5 58 0)
+	(gr_text "LED"
+		(at 51.5 34 0)
 		(layer "F.SilkS")
 		(effects
@@
 		)
 	)
-	(gr_text "TERM: LAST DRIVE ONLY"
-		(at 42 89.5 0)
+	(gr_text "DS 4 3 2 1"
+		(at 114.3 88.2 0)
 		(layer "F.SilkS")
 		(effects
 			(font
-				(size 0.9 0.9)
-				(thickness 0.135)
+				(size 0.8 0.8)
+				(thickness 0.12)
 			)
 		)
 	)
-	(gr_text "ACT"
-		(at 31.6 62 90)
+	(gr_text "RST"
+		(at 160.5 58 0)
 		(layer "F.SilkS")
 		(effects
@@
 		)
 	)
-	(gr_text "PWR"
-		(at 31.6 56 90)
+	(gr_text "ACT"
+		(at 31.6 62 90)
 		(layer "F.SilkS")
 		(effects
@@
 		)
 	)
-	(gr_text "DS 4 3 2 1"
-		(at 114.3 88.2 0)
+	(gr_text "J2 DATA"
+		(at 151.45 96.3 0)
 		(layer "F.SilkS")
 		(effects
 			(font
-				(size 0.8 0.8)
-				(thickness 0.12)
+				(size 1 1)
+				(thickness 0.15)
+			)
+		)
+	)
+	(gr_text "FIRMWARE: github.com/kuba2k2/pico506"
+		(at 89 54.2 0)
+		(layer "B.SilkS")
+		(effects
+			(font
+				(size 1 1)
+				(thickness 0.15)
 			)
+			(justify mirror)
 		)
 	)
-	(gr_text "github.com/kuba2k2/pico506"
-		(at 89 53.5 0)
+	(gr_text "github.com/hmerrett/pico506-pcb"
+		(at 89 52 0)
 		(layer "B.SilkS")
 		(effects
@@
 	)
 	(gr_text "PICO506  REV 1.0"
-		(at 89 50 0)
+		(at 89 49 0)
 		(layer "B.SilkS")
 		(effects
@@
 		)
 	)
-	(gr_text "FAB: 1.6mm FR4, 1oz Cu. Card edge fingers hard gold (Ni 2.5um min / Au 0.4um min), bevel 30deg both card edges."
-		(at 99 108.5 0)
+	(gr_text "Key slots 0.91mm routed through. Board rear edge = drive rear plane; tabs protrude 5mm for cable access."
+		(at 99 111 0)
 		(layer "Cmts.User")
 		(effects
@@
 		)
 	)
-	(gr_text "Key slots 0.91mm routed through. Board rear edge = drive rear plane; tabs protrude 5mm for cable access."
-		(at 99 111 0)
+	(gr_text "FAB: 1.6mm FR4, 1oz Cu. Card edge fingers hard gold (Ni 2.5um min / Au 0.4um min), bevel 30deg both card edges."
+		(at 99 108.5 0)
 		(layer "Cmts.User")
 		(effects
@@
 		(polygon
 			(pts
-				(xy 137.5 96.8) (xy 165.4 96.8) (xy 165.4 110) (xy 137.5 110)
+				(xy 61.255 96.8) (xy 106.945 96.8) (xy 106.945 110) (xy 61.255 110)
 			)
 		)
@@
 		(polygon
 			(pts
-				(xy 61.255 96.8) (xy 106.945 96.8) (xy 106.945 110) (xy 61.255 110)
+				(xy 137.5 96.8) (xy 165.4 96.8) (xy 165.4 110) (xy 137.5 110)
 			)
 		)
